Commit message: motor_control node added

File: vision_bot/urdf/vision_bot_qr.urdf (robot description, URDF)
Before this commit: robot vision_bot, 8 links, 7 joints
Joints:
- joint camera_joint: origin xyz=0 -0.18 0.2 rpy=0 0.0 -1.57 -> xyz=0 -0.18 0.2 rpy=0.0 0 -1.57

Commit message: Ready for Recording

File: vision_bot/urdf/vision_bot_qr.urdf (robot description, URDF)
Before this commit: robot vision_bot, 8 links, 7 joints
Links:
- added link lidar
Joints:
- added joint lidar_joint: type fixed, parent base_link, child lidar, origin xyz=0 -0.23 0.1 rpy=0.0 0 3.14, axis 0.0 0.0 1.0
